File: botao_colibri/power_management.kicad_sch (KiCad schematic)
At the start: 24 parts, among them J1 USB4970-00-A_REVA, J3 Conn_01x02, SW1 B3F-3122, U4 NPM1300-QEAA-R7

Commit message: continuação
Parts:
- added GND1: TestPoint, TestPoint:TestPoint_Pad_D1.0mm, symbol Connector:TestPoint
Connections:
- net GND: now also GND1.1
Changed lines of the file:
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@@
 	)
 	(junction
-		(at 194.31 82.55)
+		(at 184.15 105.41)
 		(diameter 0)
 		(color 0 0 0 0)
 	)
 	(junction
-		(at 123.19 33.02)
+		(at 194.31 82.55)
 		(diameter 0)
 		(color 0 0 0 0)
 	)
 	(junction
-		(at 184.15 105.41)
+		(at 123.19 33.02)
 		(diameter 0)
 		(color 0 0 0 0)
@@
 	)
 	(junction
+		(at 226.06 116.84)
+		(diameter 0)
+		(color 0 0 0 0)
+	)
+	(junction
 		(at 161.29 80.01)
 		(diameter 0)
@@
 		)
 		(property "Value" "+BATT"
-			(at 191.77 103.632 0)
+			(at 188.976 102.108 0)
 			(show_name no)
 			(do_not_autoplace no)
@@
 					(unit 1)
 				)
+			)
+		)
+	)
+	(symbol
+		(lib_id "Connector:TestPoint")
+		(at 226.06 116.84 180)
+		(unit 1)
+		(body_style 1)
+		(exclude_from_sim no)
+		(in_bom yes)
+		(on_board yes)
+		(in_pos_files yes)
+		(dnp no)
+		(property "Reference" "GND1"
+			(at 231.648 120.396 0)
+			(show_name no)
+			(do_not_autoplace no)
+			(effects
+				(font
+					(size 1.27 1.27)
+				)
+				(justify left)
+			)
+		)
+		(property "Value" "TestPoint"
+			(at 236.22 119.888 0)
+			(hide yes)
+			(show_name no)
+			(do_not_autoplace no)
+			(effects
+				(font
+					(size 1.27 1.27)
+				)
+				(justify left)
+			)
+		)
+		(property "Footprint" "TestPoint:TestPoint_Pad_D1.0mm"
+			(at 220.98 116.84 0)
+			(hide yes)
+			(show_name no)
+			(do_not_autoplace no)
+			(effects
+				(font
+					(size 1.27 1.27)
+				)
+			)
+		)
+		(property "Datasheet" ""
+			(at 220.98 116.84 0)
+			(hide yes)
+			(show_name no)
+			(do_not_autoplace no)
+			(effects
+				(font
+					(size 1.27 1.27)
+				)
+			)
+		)
+		(property "Description" "test point"
+			(at 226.06 116.84 0)
+			(hide yes)
+			(show_name no)
+			(do_not_autoplace no)
+			(effects
+				(font
+					(size 1.27 1.27)
+				)
+			)
+		)
+		(pin "1"
+		)
+		(instances
+			(project "colibri_pcb_qfn"
+				(path "/e8a5d668-2ab0-4e4a-af8f-1266e6d31156"
+					(reference "GND1")
+					(unit 1)
+				)
