File: botao_colibri/colibri_pcb_qfn.kicad_pcb (KiCad board)
At the start: 2 copper layers, 72.5 x 47.1 mm, 45 parts, among them J1 USB4970-00-A_REVA, J2 TC2030, J4 PJ-307C, J5 Conn_01x06, J6 Conn_01x06, J7 Conn_01x02, J8 Conn_01x02, SW1 B3F-3122, U1 ME54BS12, U4 NPM1300-QEAA-R7

Commit message: Acabamentos
Parts:
- P1.02 P1.09 P1.10 P2.00 P1.08 P1.07: renamed from J6
- P2.01 P2.03 P2.02 P2.05 P2.08 P2.06: renamed from J5
- moved P2.01 P2.03 P2.02 P2.05 P2.08 P2.06 1.05 mm to (128.2, 112.6)
- moved P1.02 P1.09 P1.10 P2.00 P1.08 P1.07 0.87 mm to (128.1, 109.0)
- renumbered J8 to BATT_CONN, J7 to GND_VDD, D1 to LED_RGB, sw_principal1 to MAIN_SWITCH, J4 to P2_CONN, SW1 to SWITCH, J2 to TC2030, J1 to USB_C
Routing:
- net P2.02: track 52.9 -> 57.1 mm
- net BTN_PWR: track 37.6 -> 33.9 mm, vias 2 -> 1
- net PVDD: track 36.4 -> 38.1 mm
- net P2.05: track 59.1 -> 57.7 mm
- net P2.08: track 61.7 -> 62.8 mm
- net P2.06: track 76.6 -> 77.7 mm
- net P1.07: track 42.2 -> 43.1 mm
- net P1.10: track 25.2 -> 24.3 mm
- net P1.09: track 23.5 -> 22.7 mm
- net P2.00: track 27.3 -> 26.4 mm
- net P1.08: track 21.9 -> 21.3 mm
