File: botao_colibri/_restore_backup_2026-09-03T15-52-00-749/colibri_pcb_qfn.kicad_pcb (KiCad board)
At the start: 2 copper layers, 72.5 x 47.1 mm, 45 parts, among them J1 USB4970-00-A_REVA, J2 TC2030, J4 PJ-307C, J5 Conn_01x06, J6 Conn_01x06, J7 Conn_01x02, J8 Conn_01x02, SW1 B3F-3122, U1 ME54BS12, U4 NPM1300-QEAA-R7

Commit message: Pedidos do henrique
Parts:
- moved VBATT_TP1 10.8 mm to (186.0, 111.4)
- moved J8 5.26 mm to (189.5, 107.3), turned to 90 degrees
- moved R1 4.51 mm to (186.4, 108.5)
- moved D1 3.00 mm to (192.8, 115.6)
- moved C3 2.60 mm to (186.4, 103.5)
- moved GND1 1.27 mm to (193.4, 111.4)
- moved C8 0.85 mm to (187.0, 99.6)
- moved J3 0.68 mm to (189.8, 111.4)
- renumbered -BATT to GND1, +BATT to J3
Connections:
- J8 pad 1: +BATT -> BATT+
Routing:
- net +BATT: track 29.8 -> 9.79 mm
- net GND: track 254.4 -> 237.1 mm
- net Net-(D1-Pad3): track 24.5 -> 20.6 mm
- net Net-(D1-Pad1): track 31.7 -> 28.5 mm
- net VDD: track 138.8 -> 135.9 mm
- net I2C_SCL: track 85.6 -> 88.2 mm
- net Net-(D1-Pad2): track 18.8 -> 16.7 mm, vias 2 -> 0
- net Net-(U4-VSET1): track 14.0 -> 12.8 mm
